File: dogcage_kicad/dogcage.sch (KiCad schematic (older format))
At the start: 18 parts, among them CON1 BARREL_JACK, M1 XBEE, P1 Door Sensor, P2 Servo, P3 CONN_01X10, P4 CONN_01X10, P5 CONN_01X14, P6 CONN_01X05, P7 CONN_01X14, Q1 TIP120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

Commit message: Routing complete
Parts:
- removed P6: CONN_01X05, Pin_Headers:Pin_Header_Straight_1x05, symbol CONN_01X05
Connections:
- net XBEE_CTL: now also M1.4 (DIO12/SPI_MISO), P3.4 (P4), P7.4 (P4), U2.30 (23); no longer M1.9 (DIO8/DTR#/SLEEP_RQ), P3.9 (P9), P7.14 (P14), U2.20 (13)
- net at P5.12 (P12), U2.12 (10): no longer P1.1 (P1)
- net at P5.13 (P13), U2.13 (11): now also SW1.1
- net at P5.14 (P14), U2.14 (12): now also P1.1 (P1); no longer Q1.1 (B)
- net at U2.19 (26): now also Q1.1 (B)
- net at P7.12 (P12), U2.22 (15): no longer SW1.1
- new net: P7.14 (P14), U2.20 (13)
- new net: M1.9 (DIO8/DTR#/SLEEP_RQ), P3.9 (P9)
- no-connect marks 1 -> 4
Other:
- moved on the sheet: SW1
Changed lines of the file:
@@
 L GND #PWR03
 U 1 1 553C47AE
-P 8850 3800
-F 0 "#PWR03" H 8850 3550 50  0001 C CNN
-F 1 "GND" H 8850 3650 50  0000 C CNN
-F 2 "" H 8850 3800 60  0000 C CNN
-F 3 "" H 8850 3800 60  0000 C CNN
-	1    8850 3800
+P 5750 3800
+F 0 "#PWR03" H 5750 3550 50  0001 C CNN
+F 1 "GND" H 5750 3650 50  0000 C CNN
+F 2 "" H 5750 3800 60  0000 C CNN
+F 3 "" H 5750 3800 60  0000 C CNN
+	1    5750 3800
 	1    0    0    -1
 $EndComp
@@
 	7450 4950 7450 5150
 Wire Wire Line
-	7300 3950 7750 3950
-Wire Wire Line
-	6650 2600 6650 4750
+	7450 3950 7750 3950
 Wire Wire Line
 	7450 4550 7450 4150
@@
 	7450 4150 7750 4150
 Wire Wire Line
-	4250 1150 4450 1150
-Wire Wire Line
-	4450 1150 4800 1150
+	4250 1150 4800 1150
 Wire Wire Line
 	4800 1150 4800 1000
 Wire Wire Line
-	3850 1450 3850 1600
-Wire Wire Line
-	3850 1600 3850 1700
+	3850 1450 3850 1700
 Wire Wire Line
 	3250 1550 3250 1600
 Wire Wire Line
-	3250 1600 3850 1600
-Wire Wire Line
-	3850 1600 4450 1600
+	3250 1600 4450 1600
 Connection ~ 3850 1600
 Wire Wire Line
@@
 	2950 1000 2950 1150
 Wire Wire Line
-	2950 1150 3250 1150
-Wire Wire Line
-	3250 1150 3450 1150
+	2950 1150 3450 1150
 Wire Wire Line
 	3250 1250 3250 1150
@@
 $EndComp
 Wire Wire Line
-	1500 2950 1750 2950
-Wire Wire Line
-	1750 2950 1950 2950
+	1500 2950 1950 2950
 Wire Wire Line
 	1500 3050 1950 3050
@@
 $EndComp
 Wire Wire Line
-	3750 3450 4000 3450
-Wire Wire Line
-	4000 3450 4300 3450
+	3750 3450 4300 3450
 Wire Wire Line
 	4000 3450 4000 4050
@@
 $EndComp
 Wire Wire Line
-	6350 2400 6350 3350
-Wire Wire Line
-	6050 2400 6350 2400
-Wire Wire Line
-	6350 2400 6650 2400
-Wire Wire Line
-	6650 2600 6050 2600
-Wire Wire Line
-	6650 2500 6050 2500
+	6050 2400 6650 2400
+Wire Wire Line
+	6050 2600 6650 2600
+Wire Wire Line
+	6050 2500 6650 2500
 Wire Wire Line
 	6650 2300 6050 2300
@@
 	6650 1400 6050 1400
 Wire Wire Line
-	8650 2400 8850 2400
-Wire Wire Line
-	8850 2400 9100 2400
-Wire Wire Line
-	8850 3050 8850 2400
-Connection ~ 8850 2400
+	8650 2400 9100 2400
 Wire Wire Line
 	8650 2500 9100 2500
@@
 	8650 1400 9100 1400
 Wire Wire Line
-	8650 1300 8850 1300
-Wire Wire Line
-	8850 1300 9100 1300
+	8650 1300 9100 1300
 Connection ~ 8850 1300
 Wire Wire Line
-	8850 3800 8850 3650
-$Comp
-L CONN_01X05 P6
-U 1 1 55454EDE
-P 7650 3400
-F 0 "P6" H 7650 3700 50  0000 C CNN
-F 1 "CONN_01X05" V 7750 3400 50  0000 C CNN
-F 2 "Pin_Headers:Pin_Header_Straight_1x05" H 7650 3400 60  0001 C CNN
-F 3 "" H 7650 3400 60  0000 C CNN
-	1    7650 3400
-	0    1    1    0
-$EndComp
-Wire Wire Line
-	6650 4750 7150 4750
-Wire Wire Line
-	7450 3100 7450 3150
-Wire Wire Line
-	7450 3150 7450 3200
-Wire Wire Line
-	7450 3150 7300 3150
-Wire Wire Line
-	7300 3150 7300 3950
-Connection ~ 7450 3150
-Wire Wire Line
-	7550 3100 7550 3200
-Wire Wire Line
-	7650 3100 7650 3200
-Wire Wire Line
-	7750 3100 7750 3200
-Wire Wire Line
-	7850 3100 7850 3200
-Wire Wire Line
-	1500 3850 1750 3850
-Wire Wire Line
-	1750 3850 1950 3850
+	5750 3800 5750 3650
+Wire Wire Line
+	7450 3100 7450 3950
+Wire Wire Line
+	1500 3850 1950 3850
 Wire Wire Line
 	1750 3850 1750 4050
 Connection ~ 1750 3850
 Wire Wire Line
-	6050 1300 6350 1300
-Wire Wire Line
-	6350 1300 6650 1300
+	6050 1300 6650 1300
 Wire Wire Line
 	6350 1300 6350 950
@@
 	5550 950  5550 1450
 Connection ~ 6350 1300
-Connection ~ 6350 2400
 $Comp
 L SW_PUSH SW1
 U 1 1 553C46F2
-P 8850 3350
-F 0 "SW1" H 9000 3460 50  0000 C CNN
-F 1 "SW_PUSH" H 8850 3270 50  0000 C CNN
-F 2 "Buttons_Switches_ThroughHole:SW_PUSH_SMALL" H 8850 3350 60  0001 C CNN
-F 3 "" H 8850 3350 60  0000 C CNN
-	1    8850 3350
-	0    1    1    0
-$EndComp
-Text Label 8650 2600 0    60   ~ 0
+P 5750 3350
+F 0 "SW1" H 5900 3460 50  0000 C CNN
+F 1 "SW_PUSH" H 5750 3270 50  0000 C CNN
+F 2 "Buttons_Switches_ThroughHole:SW_PUSH_SMALL" H 5750 3350 60  0001 C CNN
+F 3 "" H 5750 3350 60  0000 C CNN
+	1    5750 3350
+	0    -1   1    0
+$EndComp
+NoConn ~ 7550 3100
+NoConn ~ 7650 3100
+NoConn ~ 7750 3100
+Wire Wire Line
+	7850 3100 7850 3500
+Wire Wire Line
+	7850 3500 6850 3500
+Wire Wire Line
+	6850 3500 6850 4750
+Wire Wire Line
+	6850 4750 7150 4750
+Wire Wire Line
+	5750 3050 6300 3050
+Wire Wire Line
+	6300 3050 6300 2500
+Connection ~ 6300 2500
+Wire Wire Line
+	6350 3350 6350 2600
+Connection ~ 6350 2600
+Text Label 1500 3250 0    60   ~ 0
 XBEE_CTL
-Text Label 1500 3750 0    60   ~ 0
+Text Label 8650 1600 0    60   ~ 0
 XBEE_CTL
 $EndSCHEMATC
