File: hw/dogcage.sch (KiCad schematic (older format))
At the start: 23 parts, among them CON1 BARREL_JACK, P1 Door, P2 Lock, Q1 TIP120, Q2 TIP120, SW1 SW_PUSH, SW2 SW_PUSH, U1 LD1117S50TR, U2 LD1117S33TR, U3 TEENSYLC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

Commit message: Switched to non-polarized caps on regulators
Parts:
- removed C1: .1uF, Capacitors_Elko_ThroughHole:Elko_vert_11x5mm_RM2, symbol CP
- removed C2, C3: 10uF, Capacitors_Elko_ThroughHole:Elko_vert_11x5mm_RM2, symbol CP
- added C1: .1uF, symbol C
- added C2, C3: 10uF, symbol C
Changed lines of the file:
@@
-$EndComp
-$Comp
-L CP C2
-U 1 1 553C53E8
-P 4000 1400
-F 0 "C2" H 4025 1500 50  0000 L CNN
-F 1 "10uF" H 4025 1300 50  0000 L CNN
-F 2 "Capacitors_Elko_ThroughHole:Elko_vert_11x5mm_RM2" H 4038 1250 30  0001 C CNN
-F 3 "" H 4000 1400 60  0000 C CNN
-	1    4000 1400
-	1    0    0    -1
-$EndComp
-$Comp
-L CP C3
-U 1 1 553C5452
-P 5350 1400
-F 0 "C3" H 5375 1500 50  0000 L CNN
-F 1 "10uF" H 5375 1300 50  0000 L CNN
-F 2 "Capacitors_Elko_ThroughHole:Elko_vert_11x5mm_RM2" H 5388 1250 30  0001 C CNN
-F 3 "" H 5350 1400 60  0000 C CNN
-	1    5350 1400
-	1    0    0    -1
 $EndComp
 $Comp
@@
 F 3 "" H 3300 1700 60  0000 C CNN
 	1    3300 1700
-	1    0    0    -1
-$EndComp
-$Comp
-L CP C1
-U 1 1 55A16AFB
-P 2750 1400
-F 0 "C1" H 2775 1500 50  0000 L CNN
-F 1 ".1uF" H 2775 1300 50  0000 L CNN
-F 2 "Capacitors_Elko_ThroughHole:Elko_vert_11x5mm_RM2" H 2788 1250 30  0001 C CNN
-F 3 "" H 2750 1400 60  0000 C CNN
-	1    2750 1400
 	1    0    0    -1
 $EndComp
@@
 Wire Wire Line
 	8900 4150 9150 4150
+$Comp
+L C C1
+U 1 1 55AB32EC
+P 2750 1400
+F 0 "C1" H 2775 1500 50  0000 L CNN
+F 1 ".1uF" H 2775 1300 50  0000 L CNN
+F 2 "" H 2788 1250 30  0000 C CNN
+F 3 "" H 2750 1400 60  0000 C CNN
+	1    2750 1400
+	1    0    0    -1
+$EndComp
+$Comp
+L C C2
+U 1 1 55AB35B2
+P 4000 1400
+F 0 "C2" H 4025 1500 50  0000 L CNN
+F 1 "10uF" H 4025 1300 50  0000 L CNN
+F 2 "" H 4038 1250 30  0000 C CNN
+F 3 "" H 4000 1400 60  0000 C CNN
+	1    4000 1400
+	1    0    0    -1
+$EndComp
+$Comp
+L C C3
+U 1 1 55AB367C
+P 5350 1400
+F 0 "C3" H 5375 1500 50  0000 L CNN
+F 1 "10uF" H 5375 1300 50  0000 L CNN
+F 2 "" H 5388 1250 30  0000 C CNN
+F 3 "" H 5350 1400 60  0000 C CNN
+	1    5350 1400
+	1    0    0    -1
+$EndComp
 $EndSCHEMATC

Commit message: Placement in progress
Parts:
- C1, C2, C3: footprint (none) -> Capacitors_SMD:C_0805_HandSoldering
- C4: footprint Capacitors_Elko_ThroughHole:Elko_vert_11x5mm_RM2 -> Capacitors_SMD:c_elec_3x5.3
- D2: footprint LEDs:LED-3MM -> LEDs:LED-0805
- Q1, Q2: footprint ~ -> Power_Integrations:TO-220
- R1, R2, R4, R5, R6: footprint (none) -> Resistors_SMD:R_0805_HandSoldering
- R3: footprint Resistors_ThroughHole:Resistor_Horizontal_RM10mm -> Resistors_SMD:R_0805_HandSoldering
- SW2: footprint (none) -> Buttons_Switches_ThroughHole:SW_PUSH_SMALL
- U1, U2: footprint SOT-223 -> SMD_Packages:SOT-223
- U4: footprint (none) -> ESP8266:ESP-01
Changed lines of the file:
@@
 F 0 "Q1" H 7600 4825 50  0000 L CNN
 F 1 "TIP120" H 7600 4750 50  0000 L CNN
-F 2 "~" H 7600 4675 50  0000 L CIN
+F 2 "Power_Integrations:TO-220" H 7600 4675 50  0000 L CIN
 F 3 "" H 7350 4750 50  0000 L CNN
 	1    7350 4750
@@
 F 0 "U2" H 4750 1450 40  0000 C CNN
 F 1 "LD1117S33TR" H 4750 1400 40  0000 C CNN
-F 2 "SOT-223" H 4750 1300 40  0000 C CNN
+F 2 "SMD_Packages:SOT-223" H 4750 1300 40  0000 C CNN
 F 3 "" H 4750 1200 60  0000 C CNN
 	1    4750 1200
@@
 F 0 "D2" H 4750 2850 50  0000 C CNN
 F 1 "Assoc LED" H 4750 2650 50  0000 C CNN
-F 2 "LEDs:LED-3MM" H 4750 2750 60  0001 C CNN
+F 2 "LEDs:LED-0805" H 4750 2750 60  0001 C CNN
 F 3 "" H 4750 2750 60  0000 C CNN
 	1    4750 2750
@@
 F 0 "R3" V 4830 3200 50  0000 C CNN
 F 1 "330" V 4750 3200 50  0000 C CNN
-F 2 "Resistors_ThroughHole:Resistor_Horizontal_RM10mm" V 4680 3200 30  0001 C CNN
+F 2 "Resistors_SMD:R_0805_HandSoldering" V 4680 3200 30  0001 C CNN
 F 3 "" H 4750 3200 30  0000 C CNN
 	1    4750 3200
@@
 F 0 "R5" V 7080 4500 50  0000 C CNN
 F 1 "470" V 7000 4500 50  0000 C CNN
-F 2 "" V 6930 4500 30  0000 C CNN
+F 2 "Resistors_SMD:R_0805_HandSoldering" V 6930 4500 30  0001 C CNN
 F 3 "" H 7000 4500 30  0000 C CNN
 	1    7000 4500
@@
 F 0 "Q2" H 9050 4825 50  0000 L CNN
 F 1 "TIP120" H 9050 4750 50  0000 L CNN
-F 2 "~" H 9050 4675 50  0000 L CIN
+F 2 "Power_Integrations:TO-220" H 9050 4675 50  0000 L CIN
 F 3 "" H 8800 4750 50  0000 L CNN
 	1    8800 4750
@@
 F 0 "R6" V 8580 4500 50  0000 C CNN
 F 1 "470" V 8500 4500 50  0000 C CNN
-F 2 "" V 8430 4500 30  0000 C CNN
+F 2 "Resistors_SMD:R_0805_HandSoldering" V 8430 4500 30  0001 C CNN
 F 3 "" H 8500 4500 30  0000 C CNN
 	1    8500 4500
@@
 F 0 "U1" H 3300 1450 40  0000 C CNN
 F 1 "LD1117S50TR" H 3300 1400 40  0000 C CNN
-F 2 "SOT-223" H 3300 1300 40  0000 C CNN
+F 2 "SMD_Packages:SOT-223" H 3300 1300 40  0000 C CNN
 F 3 "" H 3300 1200 60  0000 C CNN
 	1    3300 1200
@@
 F 0 "C4" H 6325 4500 50  0000 L CNN
 F 1 "100uF" H 6325 4300 50  0000 L CNN
-F 2 "Capacitors_Elko_ThroughHole:Elko_vert_11x5mm_RM2" H 6338 4250 30  0001 C CNN
+F 2 "Capacitors_SMD:c_elec_3x5.3" H 6338 4250 30  0001 C CNN
 F 3 "" H 6300 4400 60  0000 C CNN
 	1    6300 4400
@@
 F 0 "U4" H 2800 3300 50  0000 C CNN
 F 1 "ESP-01v090" H 2800 3500 50  0000 C CNN
-F 2 "" H 2800 3400 50  0001 C CNN
+F 2 "ESP8266:ESP-01" H 2800 3400 50  0001 C CNN
 F 3 "" H 2800 3400 50  0001 C CNN
 	1    2800 3400
@@
 F 0 "SW2" H 4400 3860 50  0000 C CNN
 F 1 "SW_PUSH" H 4250 3670 50  0000 C CNN
-F 2 "" H 4250 3750 60  0000 C CNN
+F 2 "Buttons_Switches_ThroughHole:SW_PUSH_SMALL" H 4250 3750 60  0001 C CNN
 F 3 "" H 4250 3750 60  0000 C CNN
 	1    4250 3750
@@
 F 0 "R1" V 4580 3000 50  0000 C CNN
 F 1 "10K" V 4500 3000 50  0000 C CNN
-F 2 "" V 4430 3000 30  0000 C CNN
+F 2 "Resistors_SMD:R_0805_HandSoldering" V 4430 3000 30  0001 C CNN
 F 3 "" H 4500 3000 30  0000 C CNN
 	1    4500 3000
@@
 F 0 "R4" V 1180 3300 50  0000 C CNN
 F 1 "10K" V 1100 3300 50  0000 C CNN
-F 2 "" V 1030 3300 30  0000 C CNN
+F 2 "Resistors_SMD:R_0805_HandSoldering" V 1030 3300 30  0001 C CNN
 F 3 "" H 1100 3300 30  0000 C CNN
 	1    1100 3300
@@
 F 0 "R2" V 1380 3200 50  0000 C CNN
 F 1 "10K" V 1300 3200 50  0000 C CNN
-F 2 "" V 1230 3200 30  0000 C CNN
+F 2 "Resistors_SMD:R_0805_HandSoldering" V 1230 3200 30  0001 C CNN
 F 3 "" H 1300 3200 30  0000 C CNN
 	1    1300 3200
@@
 F 0 "C1" H 2775 1500 50  0000 L CNN
 F 1 ".1uF" H 2775 1300 50  0000 L CNN
-F 2 "" H 2788 1250 30  0000 C CNN
+F 2 "Capacitors_SMD:C_0805_HandSoldering" H 2788 1250 30  0001 C CNN
 F 3 "" H 2750 1400 60  0000 C CNN
 	1    2750 1400
@@
 F 0 "C2" H 4025 1500 50  0000 L CNN
 F 1 "10uF" H 4025 1300 50  0000 L CNN
-F 2 "" H 4038 1250 30  0000 C CNN
+F 2 "Capacitors_SMD:C_0805_HandSoldering" H 4038 1250 30  0001 C CNN
 F 3 "" H 4000 1400 60  0000 C CNN
 	1    4000 1400
@@
 F 0 "C3" H 5375 1500 50  0000 L CNN
 F 1 "10uF" H 5375 1300 50  0000 L CNN
-F 2 "" H 5388 1250 30  0000 C CNN
+F 2 "Capacitors_SMD:C_0805_HandSoldering" H 5388 1250 30  0001 C CNN
 F 3 "" H 5350 1400 60  0000 C CNN
 	1    5350 1400

Commit message: Swapped TIP120s out for generic Darlington NPN transistors
Parts:
- removed Q1, Q2: TIP120, Power_Integrations:TO-220, symbol TIP120
- added Q1, Q2: Darl_NPN, symbol Darl_NPN
Other:
- moved on the sheet: R5, R6
Changed lines of the file:
@@
 L GND #PWR02
 U 1 1 553C464F
-P 7450 5150
-F 0 "#PWR02" H 7450 4900 50  0001 C CNN
-F 1 "GND" H 7450 5000 50  0000 C CNN
-F 2 "" H 7450 5150 60  0000 C CNN
-F 3 "" H 7450 5150 60  0000 C CNN
-	1    7450 5150
+P 7450 5250
+F 0 "#PWR02" H 7450 5000 50  0001 C CNN
+F 1 "GND" H 7450 5100 50  0000 C CNN
+F 2 "" H 7450 5250 60  0000 C CNN
+F 3 "" H 7450 5250 60  0000 C CNN
+	1    7450 5250
 	1    0    0    -1
 $EndComp
@@
 F 3 "" H 5650 3400 60  0000 C CNN
 	1    5650 3400
-	1    0    0    -1
-$EndComp
-$Comp
-L TIP120 Q1
-U 1 1 553C49B0
-P 7350 4750
-F 0 "Q1" H 7600 4825 50  0000 L CNN
-F 1 "TIP120" H 7600 4750 50  0000 L CNN
-F 2 "Power_Integrations:TO-220" H 7600 4675 50  0000 L CIN
-F 3 "" H 7350 4750 50  0000 L CNN
-	1    7350 4750
 	1    0    0    -1
 $EndComp
@@
 L R R5
 U 1 1 558214B8
-P 7000 4500
-F 0 "R5" V 7080 4500 50  0000 C CNN
-F 1 "470" V 7000 4500 50  0000 C CNN
-F 2 "Resistors_SMD:R_0805_HandSoldering" V 6930 4500 30  0001 C CNN
-F 3 "" H 7000 4500 30  0000 C CNN
-	1    7000 4500
-	1    0    0    -1
-$EndComp
-$Comp
-L TIP120 Q2
-U 1 1 559DEA4D
-P 8800 4750
-F 0 "Q2" H 9050 4825 50  0000 L CNN
-F 1 "TIP120" H 9050 4750 50  0000 L CNN
-F 2 "Power_Integrations:TO-220" H 9050 4675 50  0000 L CIN
-F 3 "" H 8800 4750 50  0000 L CNN
-	1    8800 4750
+P 6900 4500
+F 0 "R5" V 6980 4500 50  0000 C CNN
+F 1 "470" V 6900 4500 50  0000 C CNN
+F 2 "Resistors_SMD:R_0805_HandSoldering" V 6830 4500 30  0001 C CNN
+F 3 "" H 6900 4500 30  0000 C CNN
+	1    6900 4500
 	1    0    0    -1
 $EndComp
@@
 L R R6
 U 1 1 559DEC4E
-P 8500 4500
-F 0 "R6" V 8580 4500 50  0000 C CNN
-F 1 "470" V 8500 4500 50  0000 C CNN
-F 2 "Resistors_SMD:R_0805_HandSoldering" V 8430 4500 30  0001 C CNN
-F 3 "" H 8500 4500 30  0000 C CNN
-	1    8500 4500
+P 8400 4500
+F 0 "R6" V 8480 4500 50  0000 C CNN
+F 1 "470" V 8400 4500 50  0000 C CNN
+F 2 "Resistors_SMD:R_0805_HandSoldering" V 8330 4500 30  0001 C CNN
+F 3 "" H 8400 4500 30  0000 C CNN
+	1    8400 4500
 	1    0    0    -1
 $EndComp
@@
 L GND #PWR010
 U 1 1 559DEE7F
-P 8900 5150
-F 0 "#PWR010" H 8900 4900 50  0001 C CNN
-F 1 "GND" H 8900 5000 50  0000 C CNN
-F 2 "" H 8900 5150 60  0000 C CNN
-F 3 "" H 8900 5150 60  0000 C CNN
-	1    8900 5150
+P 8900 5250
+F 0 "#PWR010" H 8900 5000 50  0001 C CNN
+F 1 "GND" H 8900 5100 50  0000 C CNN
+F 2 "" H 8900 5250 60  0000 C CNN
+F 3 "" H 8900 5250 60  0000 C CNN
+	1    8900 5250
 	1    0    0    -1
 $EndComp
@@
 D2
 Wire Wire Line
-	7450 4950 7450 5150
+	7450 5050 7450 5250
 Wire Wire Line
 	7450 4550 7450 4150
@@
 	4750 2950 4750 3050
 Wire Wire Line
-	7000 4650 7000 4750
-Wire Wire Line
-	7000 4750 7150 4750
+	6900 4650 6900 4750
+Wire Wire Line
+	6900 4750 7050 4750
 Wire Wire Line
 	6300 4100 6300 4250
@@
 D12
 Wire Wire Line
-	7000 4100 7000 4350
-Text Label 7000 4300 1    60   ~ 0
+	6900 4100 6900 4350
+Text Label 6900 4300 1    60   ~ 0
 D11
 Wire Wire Line
-	8500 4100 8500 4350
-Text Label 8500 4300 1    60   ~ 0
+	8400 4100 8400 4350
+Text Label 8400 4300 1    60   ~ 0
 D12
 NoConn ~ 6650 2100
@@
 NoConn ~ 6650 1700
 Wire Wire Line
-	8500 4650 8500 4750
-Wire Wire Line
-	8500 4750 8600 4750
+	8400 4650 8400 4750
+Wire Wire Line
+	8400 4750 8500 4750
 Wire Wire Line
 	3300 1450 3300 1700
@@
 Connection ~ 2050 1350
 Wire Wire Line
-	8900 4950 8900 5150
+	8900 5050 8900 5250
 Wire Wire Line
 	8900 4550 8900 4150
@@
 	1    0    0    -1
 $EndComp
+$Comp
+L Darl_NPN Q1
+U 1 1 55B3E58A
+P 7300 4750
+F 0 "Q1" H 7300 4950 50  0000 C CNN
+F 1 "Darl_NPN" H 7100 4600 50  0000 C CNN
+F 2 "" H 7300 4700 60  0000 C CNN
+F 3 "" H 7300 4700 60  0000 C CNN
+	1    7300 4750
+	1    0    0    -1
+$EndComp
+$Comp
+L Darl_NPN Q2
+U 1 1 55B3EB3C
+P 8750 4750
+F 0 "Q2" H 8750 4950 50  0000 C CNN
+F 1 "Darl_NPN" H 8550 4600 50  0000 C CNN
+F 2 "" H 8750 4700 60  0000 C CNN
+F 3 "" H 8750 4700 60  0000 C CNN
+	1    8750 4750
+	1    0    0    -1
+$EndComp

Commit message: Changed NPN and button footprints to SMD
Parts:
- Q1, Q2: footprint (none) -> SMD_Packages:DPAK-2
- SW1, SW2: footprint Buttons_Switches_ThroughHole:SW_PUSH_SMALL -> Buttons_Switches_SMD:SW_SPST_FSMSM
Changed lines of the file:
@@
 F 0 "SW1" H 5800 3010 50  0000 C CNN
 F 1 "SW_PUSH" H 5650 2820 50  0000 C CNN
-F 2 "Buttons_Switches_ThroughHole:SW_PUSH_SMALL" H 5650 2900 60  0001 C CNN
+F 2 "Buttons_Switches_SMD:SW_SPST_FSMSM" H 5650 2900 60  0001 C CNN
 F 3 "" H 5650 2900 60  0000 C CNN
 	1    5650 2900
@@
 F 0 "SW2" H 4400 3860 50  0000 C CNN
 F 1 "SW_PUSH" H 4250 3670 50  0000 C CNN
-F 2 "Buttons_Switches_ThroughHole:SW_PUSH_SMALL" H 4250 3750 60  0001 C CNN
+F 2 "Buttons_Switches_SMD:SW_SPST_FSMSM" H 4250 3750 60  0001 C CNN
 F 3 "" H 4250 3750 60  0000 C CNN
 	1    4250 3750
@@
 F 0 "Q1" H 7300 4950 50  0000 C CNN
 F 1 "Darl_NPN" H 7100 4600 50  0000 C CNN
-F 2 "" H 7300 4700 60  0000 C CNN
+F 2 "SMD_Packages:DPAK-2" H 7300 4700 60  0001 C CNN
 F 3 "" H 7300 4700 60  0000 C CNN
 	1    7300 4750
@@
 F 0 "Q2" H 8750 4950 50  0000 C CNN
 F 1 "Darl_NPN" H 8550 4600 50  0000 C CNN
-F 2 "" H 8750 4700 60  0000 C CNN
+F 2 "SMD_Packages:DPAK-2" H 8750 4700 60  0001 C CNN
 F 3 "" H 8750 4700 60  0000 C CNN
 	1    8750 4750

Commit message: Moved servo power control GPIOs to other side of the Teensy
Connections:
- net labels added: D14, D15
- net labels removed: D11, D12
Changed lines of the file:
@@
 Wire Wire Line
 	5650 2400 5650 2600
-Wire Wire Line
-	6650 2500 6200 2500
-Wire Wire Line
-	6650 2600 6200 2600
 Text Label 6350 2400 0    60   ~ 0
 D10
-Text Label 6350 2500 0    60   ~ 0
-D11
-Text Label 6350 2600 0    60   ~ 0
-D12
 Wire Wire Line
 	6900 4100 6900 4350
 Text Label 6900 4300 1    60   ~ 0
-D11
+D14
 Wire Wire Line
 	8400 4100 8400 4350
 Text Label 8400 4300 1    60   ~ 0
-D12
+D15
 NoConn ~ 6650 2100
 NoConn ~ 6650 2000
@@
 NoConn ~ 6650 2300
 NoConn ~ 7850 3100
-NoConn ~ 8650 2500
-NoConn ~ 8650 2400
 NoConn ~ 8650 2300
 NoConn ~ 8650 2200
@@
 	1    0    0    -1
 $EndComp
+NoConn ~ 6650 2600
+NoConn ~ 6650 2500
+Wire Wire Line
+	8650 2500 9000 2500
+Wire Wire Line
+	8650 2400 9000 2400
+Text Label 8800 2400 0    60   ~ 0
+D15
+Text Label 8800 2500 0    60   ~ 0
+D14
 $EndSCHEMATC

Commit message: Changed barrel jack footprint to have round througholes
Parts:
- CON1: footprint Connect:BARREL_JACK -> modules:BARREL_JACK-ROUND_TH
- SW1: footprint Buttons_Switches_SMD:SW_SPST_FSMSM -> Buttons_Switches_ThroughHole:SW_PUSH_SMALL
Changed lines of the file:
@@
 F 0 "CON1" H 1400 1500 60  0000 C CNN
 F 1 "BARREL_JACK" H 1400 1050 60  0000 C CNN
-F 2 "Connect:BARREL_JACK" H 1400 1250 60  0001 C CNN
+F 2 "modules:BARREL_JACK-ROUND_TH" H 1400 1250 60  0001 C CNN
 F 3 "" H 1400 1250 60  0000 C CNN
 	1    1400 1250
@@
 F 0 "SW1" H 5800 3010 50  0000 C CNN
 F 1 "SW_PUSH" H 5650 2820 50  0000 C CNN
-F 2 "Buttons_Switches_SMD:SW_SPST_FSMSM" H 5650 2900 60  0001 C CNN
+F 2 "Buttons_Switches_ThroughHole:SW_PUSH_SMALL" H 5650 2900 60  0001 C CNN
 F 3 "" H 5650 2900 60  0000 C CNN
 	1    5650 2900

Commit message: Placement is essentially done
Parts:
- CON1: value BARREL_JACK -> 6.5V+
Changed lines of the file:
@@
 P 1400 1250
 F 0 "CON1" H 1400 1500 60  0000 C CNN
-F 1 "BARREL_JACK" H 1400 1050 60  0000 C CNN
+F 1 "6.5V+" H 1400 1050 60  0000 C CNN
 F 2 "modules:BARREL_JACK-ROUND_TH" H 1400 1250 60  0001 C CNN
 F 3 "" H 1400 1250 60  0000 C CNN

Commit message: Partially routed
Parts:
- SW1: value SW_PUSH -> Activate
- U3: value TEENSYLC -> Teensy LC
- U4: value ESP-01v090 -> ESP8266
Connections:
- net labels removed: D10
- wire segments 77 -> 76
Other:
- moved on the sheet: SW1
Changed lines of the file:
@@
 P 7650 1950
 F 0 "U3" H 7650 1850 50  0000 C CNN
-F 1 "TEENSYLC" H 7650 2050 50  0000 C CNN
+F 1 "Teensy LC" H 7650 2050 50  0000 C CNN
 F 2 "modules:Teensy-3.1" H 7650 1950 50  0001 C CNN
 F 3 "DOCUMENTATION" H 7650 1950 50  0001 C CNN
@@
 L GND #PWR03
 U 1 1 553C47AE
-P 5650 3400
-F 0 "#PWR03" H 5650 3150 50  0001 C CNN
-F 1 "GND" H 5650 3250 50  0000 C CNN
-F 2 "" H 5650 3400 60  0000 C CNN
-F 3 "" H 5650 3400 60  0000 C CNN
-	1    5650 3400
+P 8700 3300
+F 0 "#PWR03" H 8700 3050 50  0001 C CNN
+F 1 "GND" H 8700 3150 50  0000 C CNN
+F 2 "" H 8700 3300 60  0000 C CNN
+F 3 "" H 8700 3300 60  0000 C CNN
+	1    8700 3300
 	1    0    0    -1
 $EndComp
@@
 L SW_PUSH SW1
 U 1 1 553C46F2
-P 5650 2900
-F 0 "SW1" H 5800 3010 50  0000 C CNN
-F 1 "SW_PUSH" H 5650 2820 50  0000 C CNN
-F 2 "Buttons_Switches_ThroughHole:SW_PUSH_SMALL" H 5650 2900 60  0001 C CNN
-F 3 "" H 5650 2900 60  0000 C CNN
-	1    5650 2900
-	0    -1   1    0
+P 8400 3100
+F 0 "SW1" H 8550 3210 50  0000 C CNN
+F 1 "Activate" H 8400 3020 50  0000 C CNN
+F 2 "Buttons_Switches_ThroughHole:SW_PUSH_SMALL" H 8400 3100 60  0001 C CNN
+F 3 "" H 8400 3100 60  0000 C CNN
+	1    8400 3100
+	-1   0    0    -1
 $EndComp
 $Comp
@@
 P 2800 3400
 F 0 "U4" H 2800 3300 50  0000 C CNN
-F 1 "ESP-01v090" H 2800 3500 50  0000 C CNN
+F 1 "ESP8266" H 2800 3500 50  0000 C CNN
 F 2 "ESP8266:ESP-01" H 2800 3400 50  0001 C CNN
 F 3 "" H 2800 3400 50  0001 C CNN
@@
 Connection ~ 8850 1300
 Wire Wire Line
-	5650 3400 5650 3200
-Wire Wire Line
 	7450 3100 7450 3250
 Wire Wire Line
@@
 Wire Wire Line
 	8850 1400 8850 1500
-Wire Wire Line
-	6650 2400 5650 2400
-Wire Wire Line
-	5650 2400 5650 2600
-Text Label 6350 2400 0    60   ~ 0
-D10
 Wire Wire Line
 	6900 4100 6900 4350
@@
 NoConn ~ 6650 2200
 NoConn ~ 6650 2300
-NoConn ~ 7850 3100
 NoConn ~ 8650 2300
 NoConn ~ 8650 2200
@@
 Text Label 8800 2500 0    60   ~ 0
 D14
+NoConn ~ 6650 2400
+Wire Wire Line
+	7850 3100 8100 3100
+Wire Wire Line
+	8700 3100 8700 3300
 $EndSCHEMATC
